Commit message: add robot_setup_joints

File: drone_bringup/configuration_files/fixed_joint.urdf (robot description, URDF)
Before this commit: robot drone_fixed_joint, 5 links, 4 joints
Links:
- removed link elp_left_optical_frame
- removed link elp_right_optical_frame
Joints:
- removed joint elp_left_link
- removed joint elp_right_link
- removed joint r200_link
